Commit message: Updated description to contain lidar

File: brum_description/urdf/brum.urdf.xacro (robot description, xacro)
@@ -3,10 +3,10 @@
   <xacro:arg name="prefix" default="" />
   <xacro:include filename="brum_base.urdf" />
-  <xacro:include
-    filename="$(find mirte_control)/ros2_control/diffbot.ros2_control.xacro" />
-  <xacro:include
-    filename="$(find mirte_modular_hardware_interface)/urdf/joint_encoder.ros2_control.xacro" />
-  <xacro:diffbot_ros2_control
-    name="MirteHardware" prefix="$(arg prefix)" />
-  <xacro:mirte_modular_hardware_joint_encoder name="right_wheel_joint" topic="io/encoder/right" />
+  <!-- <xacro:include
+    filename="$(find mirte_control)/ros2_control/diffbot.ros2_control.xacro" /> -->
+  <!-- <xacro:include
+    filename="$(find mirte_modular_hardware_interface)/urdf/joint_encoder.ros2_control.xacro" /> -->
+  <!-- <xacro:diffbot_ros2_control
+    name="MirteHardware" prefix="$(arg prefix)" /> -->
+  <!-- <xacro:mirte_modular_hardware_joint_encoder name="right_wheel_joint" topic="io/encoder/right" /> -->
 </robot>

File: brum_description/urdf/brum_base.urdf (robot description, URDF)
Before this commit: robot brum_description, 10 links, 9 joints
Links:
- added link laser_link, mass 0.061052; collision mesh filename=package://brum_description/meshes/laser_link.STL; visual mesh filename=package://brum_description/meshes/laser_link.STL
- link caster_link: mass 0 -> 0.0062086
- link frame_link: mass 0.26203100747214 -> 0.26172
Joints:
- added joint laser_joint: type fixed, parent frame_link, child laser_link, origin xyz=0.017449 0 0.08845 rpy=-1.5708 0 -1.5708, axis 0 0 0
- joint camera_mount_joint: origin xyz=0.163248855994184 0.0767499999979599 0.0349999999999995 rpy=1.5707963267949 0 -1.5707963267949 -> xyz=0.0534488559945167 0.0262499999959915 0.0349999999999993 rpy=1.5707963267949 0 -1.5707963267949
- joint caster_joint: origin xyz=-0.018201 0.0505 -0.0442 rpy=-1.5708 0 -1.5708 -> xyz=-0.128 0 -0.032 rpy=-1.5708 0 -1.5708
- joint left_wheel_joint: axis 0 0 -1 -> 0 0 1; origin xyz=0.1098 0.12975 -0.01815 rpy=-1.5708 0 0 -> xyz=0 0.07925 -0.01815 rpy=-1.5708 0 0
- joint powerbank_joint: origin xyz=0.016919 0.0505 -0.029 rpy=-1.5708 0 -1.5708 -> xyz=-0.092881 0 -0.029 rpy=-1.5708 0 -1.5708
- joint right_wheel_joint: axis 0 0 1 -> 0 0 -1; origin xyz=0.1098 -0.02875 -0.01815 rpy=1.5708 0 0 -> xyz=0 -0.07925 -0.01815 rpy=1.5708 0 0
- joint under_cairrage_joint: origin xyz=0.1582 0.013 -0.02385 rpy=1.5708 0 1.5708 -> xyz=0.0484 -0.0375 -0.02385 rpy=1.5708 0 1.5708

Commit message: Cleanup brum_description

File: brum_description/urdf/brum.urdf.xacro (robot description, xacro)
@@ -2,5 +2,18 @@
 <robot xmlns:xacro="http://www.ros.org/wiki/xacro" name="brum">
   <xacro:arg name="prefix" default="" />
-  <xacro:include filename="brum_base.urdf" />
+  <xacro:arg name="use_lidar" default="true" />
+  <xacro:arg name="use_camera" default="true" />
+  <xacro:arg name="use_powerbank" default="true" />
+  <xacro:arg name="use_sensor_plate" default="true" />
+  <link name="base_link" />
+  <link name="base_footprint" />
+  <joint name="footprint_joint" type="fixed">
+    <parent link="base_link" />
+    <child link="base_footprint" />
+    <origin xyz="0.0 0.0 -0.0520264" />
+  </joint>
+  <xacro:include filename="$(find brum_description)/urdf/frame.urdf.xacro" ns="frame" />
+  <xacro:include filename="$(find brum_description)/urdf/wheels.urdf.xacro" />
+  <xacro:include filename="$(find brum_description)/urdf/caster.urdf.xacro" ns="caster" />
   <!-- <xacro:include
     filename="$(find mirte_control)/ros2_control/diffbot.ros2_control.xacro" /> -->
@@ -9,4 +22,18 @@
   <!-- <xacro:diffbot_ros2_control
     name="MirteHardware" prefix="$(arg prefix)" /> -->
-  <!-- <xacro:mirte_modular_hardware_joint_encoder name="right_wheel_joint" topic="io/encoder/right" /> -->
+  <!-- <xacro:mirte_modular_hardware_joint_encoder name="right_wheel_joint" topic="io/encoder/right"
+  /> -->
+  <xacro:if value="$(arg use_sensor_plate)">
+    <xacro:include filename="$(find brum_description)/urdf/sensor_plate.urdf.xacro"
+      ns="sensor_plate" />
+  </xacro:if>
+  <xacro:if value="$(arg use_powerbank)">
+    <xacro:include filename="$(find brum_description)/urdf/powerbank.urdf.xacro" />
+  </xacro:if>
+  <xacro:if value="$(arg use_camera)">
+    <xacro:include filename="$(find brum_description)/urdf/camera.urdf.xacro" ns="camera" />
+  </xacro:if>
+  <xacro:if value="$(arg use_lidar)">
+    <xacro:include filename="$(find brum_description)/urdf/lidar.urdf.xacro" />
+  </xacro:if>
 </robot>
