Commit message: Add initial gz-sim support

File: brum_description/urdf/brum.urdf.xacro (robot description, xacro)
@@ -6,4 +6,6 @@
   <xacro:arg name="use_powerbank" default="true" />
   <xacro:arg name="use_sensor_plate" default="true" />
+  <xacro:arg name="mode" default="real" />
+  <xacro:property name="mode" value="$(arg mode)" />
   <link name="base_link" />
   <link name="base_footprint" />
@@ -14,5 +16,5 @@
   </joint>
   <xacro:include filename="$(find brum_description)/urdf/frame.urdf.xacro" ns="frame" />
-  <xacro:include filename="$(find brum_description)/urdf/wheels.urdf.xacro" />
+  <xacro:include filename="$(find brum_description)/urdf/wheels.urdf.xacro" ns="wheels" />
   <xacro:include filename="$(find brum_description)/urdf/caster.urdf.xacro" ns="caster" />
   <!-- <xacro:include
@@ -37,3 +39,12 @@
     <xacro:include filename="$(find brum_description)/urdf/lidar.urdf.xacro" />
   </xacro:if>
+  <xacro:if value="${mode == 'gz-sim-diff-drive-plugin'}">
+    <gazebo>
+      <plugin filename="gz-sim-joint-state-publisher-system"
+        name="gz::sim::systems::JointStatePublisher">
+        <!-- FIXME Do not hardcode topic name -->
+        <topic>/model/brum/joint_state</topic>
+      </plugin>
+    </gazebo>
+  </xacro:if>
 </robot>

File: brum_description/urdf/camera.urdf.xacro (robot description, xacro)
@@ -1,10 +1,10 @@
 <?xml version="1.0" encoding="UTF-8"?>
 <robot xmlns:xacro="http://www.ros.org/wiki/xacro">
-  <xacro:property name="mount_width" value="0.0525"/>
-  <xacro:property name="mount_length" value="0.0135"/>
-  <xacro:property name="mount_height" value="0.032"/>
-  <xacro:property name="mount_l_offset" value="0.00475"/>
-  <xacro:property name="mount_bump_width" value="0.0145"/>
-  <xacro:property name="mount_bump_height" value="0.006"/>
+  <xacro:property name="mount_width" value="0.0525" />
+  <xacro:property name="mount_length" value="0.0135" />
+  <xacro:property name="mount_height" value="0.032" />
+  <xacro:property name="mount_l_offset" value="0.00475" />
+  <xacro:property name="mount_bump_width" value="0.0145" />
+  <xacro:property name="mount_bump_height" value="0.006" />
   <link name="camera_mount_link">
     <inertial>
@@ -36,13 +36,15 @@
     </collision> -->
     <collision>
-      <origin xyz="${mount_width/2} ${-mount_height/2} ${mount_l_offset-mount_length/2}" rpy="0.0 1.5708 1.5708"/>
+      <origin xyz="${mount_width/2} ${-mount_height/2} ${mount_l_offset-mount_length/2}"
+        rpy="0.0 1.5708 1.5708" />
       <geometry>
-        <box size="${mount_length} ${mount_width} ${mount_height}"/>
+        <box size="${mount_length} ${mount_width} ${mount_height}" />
       </geometry>
     </collision>
     <collision>
-      <origin xyz="${mount_bump_width/2} ${mount_bump_height/2} ${mount_l_offset-mount_length/2}" rpy="0.0 1.5708 1.5708"/>
+      <origin xyz="${mount_bump_width/2} ${mount_bump_height/2} ${mount_l_offset-mount_length/2}"
+        rpy="0.0 1.5708 1.5708" />
       <geometry>
-        <box size="${mount_length} ${mount_bump_width} ${mount_bump_height}"/>
+        <box size="${mount_length} ${mount_bump_width} ${mount_bump_height}" />
       </geometry>
     </collision>
@@ -55,8 +57,9 @@
     <child link="camera_mount_link" />
   </joint>
-  <xacro:property name="camera_main_width" value="0.03"/>
-  <xacro:property name="camera_plate_width" value="${camera_main_width + 0.0199}"/>
-  <xacro:property name="camera_main_thickness"  value="0.0095"/>
-  <xacro:property name="camera_plate_thickness" value="0.0030"/>
+  <xacro:property name="camera_main_width" value="0.03" />
+  <xacro:property name="camera_plate_width" value="${camera_main_width + 0.0199}" />
+  <xacro:property name="camera_main_thickness" value="0.0095" />
+  <xacro:property name="camera_plate_thickness" value="0.0030" />
+  <!-- TODO Maybe rename too center_camera and center_camera_optical-->
   <link name="camera_link">
     <inertial>
@@ -83,13 +86,13 @@
     </visual>
     <collision name="camera_main">
-      <origin xyz="${camera_main_thickness/2+camera_plate_thickness} 0.0 0.0"/>
+      <origin xyz="${camera_main_thickness/2+camera_plate_thickness} 0.0 0.0" />
       <geometry>
-        <box size="${camera_main_thickness} ${camera_main_width} ${camera_main_width}"/>
+        <box size="${camera_main_thickness} ${camera_main_width} ${camera_main_width}" />
       </geometry>
     </collision>
     <collision>
-      <origin xyz="${camera_plate_thickness/2} 0.0 0.0"/>
+      <origin xyz="${camera_plate_thickness/2} 0.0 0.0" />
       <geometry>
-        <box size="${camera_plate_thickness} ${camera_plate_width} ${camera_main_width}"/>
+        <box size="${camera_plate_thickness} ${camera_plate_width} ${camera_main_width}" />
       </geometry>
     </collision>
@@ -101,9 +104,33 @@
     <child link="camera_link" />
   </joint>
-  <link name="camera_link_optical"/>
+  <link name="camera_link_optical" />
   <joint name="camera_optical_joint" type="fixed">
-    <parent link="camera_link"/>
-    <child link="camera_link_optical"/>
-    <origin rpy="${radians(-90)} 0.0 ${radians(-90)}"/>
+    <parent link="camera_link" />
+    <child link="camera_link_optical" />
+    <origin rpy="${radians(-90)} 0.0 ${radians(-90)}" />
   </joint>
+  <xacro:if value="${mode.startswith('gz-sim')}">
+    <gazebo reference="camera_link">
+      <!-- FIXME Camera configuration -->
+      <sensor name="center_camera" type="camera">
+        <camera>
+          <horizontal_fov>1.047</horizontal_fov>
+        <image>
+          <width>320</width>
+          <height>240</height>
+        </image>
+        <clip>
+          <near>0.1</near>
+          <far>100</far>
+        </clip>
+        <optical_frame_id>camera_link_optical</optical_frame_id>
+        <camera_info_topic>center_camera/camera_info</camera_info_topic>
+      </camera>
+      <always_on>1</always_on>
+      <update_rate>25</update_rate>
+      <visualize>true</visualize>
+      <topic>center_camera/image</topic>
+    </sensor>
+  </gazebo>
+  </xacro:if>
 </robot>

File: brum_description/urdf/caster.urdf.xacro (robot description, xacro)
@@ -1,5 +1,5 @@
 <robot xmlns:xacro="http://www.ros.org/wiki/xacro">
-  <xacro:property name="ball_radius" value="0.0075"/>
-  <xacro:property name="ball_offset" value="0.005"/>
+  <xacro:property name="ball_radius" value="0.0075" />
+  <xacro:property name="ball_offset" value="0.005" />
   <link name="caster_holder_link">
     <inertial>
@@ -23,7 +23,7 @@
     </visual>
     <collision>
-      <origin xyz="0.0 ${ball_radius + ball_offset} 0.0"/>
+      <origin xyz="0.0 ${ball_radius + ball_offset} 0.0" />
       <geometry>
-        <sphere radius="${ball_radius}"/>
+        <sphere radius="${ball_radius}" />
       </geometry>
     </collision>
@@ -35,3 +35,9 @@
   </joint>
   <!-- FIXME Add roller caster_ball link-->
+  <xacro:if value="${mode.startswith('gz-sim')}">
+    <gazebo reference="caster_holder_link">
+      <mu1>0.05</mu1>
+      <mu2>0.05</mu2>
+    </gazebo>
+  </xacro:if>
 </robot>

File: brum_description/urdf/lidar.urdf.xacro (robot description, xacro)
@@ -1,9 +1,9 @@
 <?xml version="1.0" encoding="UTF-8"?>
 <robot xmlns:xacro="http://www.ros.org/wiki/xacro">
-  <xacro:property name="lidar_top_radius" value="0.0175"/>
-  <xacro:property name="lidar_top_height" value="0.0125"/>
-  <xacro:property name="lidar_top_z_offset" value="0.005"/>
-  <xacro:property name="lidar_base_height" value="0.0225"/>
-  <xacro:property name="lidar_base_width" value="0.039"/>
+  <xacro:property name="lidar_top_radius" value="0.0175" />
+  <xacro:property name="lidar_top_height" value="0.0125" />
+  <xacro:property name="lidar_top_z_offset" value="0.005" />
+  <xacro:property name="lidar_base_height" value="0.0225" />
+  <xacro:property name="lidar_base_width" value="0.039" />
   <link name="laser_mount_link">
     <inertial>
@@ -27,13 +27,14 @@
     </visual>
     <collision>
-      <origin xyz="0 ${lidar_top_z_offset-lidar_top_height/2} 0" rpy="${radians(90)} 0.0 0.0"/>
+      <origin xyz="0 ${lidar_top_z_offset-lidar_top_height/2} 0" rpy="${radians(90)} 0.0 0.0" />
       <geometry>
-        <cylinder radius="${lidar_top_radius}" length="${lidar_top_height}"/>
+        <cylinder radius="${lidar_top_radius}" length="${lidar_top_height}" />
       </geometry>
     </collision>
     <collision>
-      <origin xyz="0 ${lidar_base_height/2+lidar_top_height/2-lidar_top_z_offset/4} 0" rpy="${radians(90)} 0.0 0.0"/>
+      <origin xyz="0 ${lidar_base_height/2+lidar_top_height/2-lidar_top_z_offset/4} 0"
+        rpy="${radians(90)} 0.0 0.0" />
       <geometry>
-        <box size="${lidar_base_width} ${lidar_base_width} ${lidar_base_height}"/>
+        <box size="${lidar_base_width} ${lidar_base_width} ${lidar_base_height}" />
       </geometry>
     </collision>
@@ -50,3 +51,47 @@
     <origin rpy="1.5708 -1.5708 0.0" />
   </joint>
+  <xacro:if value="${mode.startswith('gz-sim')}">
+    <gazebo reference="laser_link">
+      <sensor name='gpu_lidar' type='gpu_lidar'>
+        <!-- <pose relative_to='brum/laser_link'>0 0 0 0 0 0</pose> -->
+        <!-- FIXME MAKE RELATIVE TO NAME  -->
+        <topic>/model/brum/laser_scan</topic>
+        <!-- <frame_id>brum/laser_link</frame_id> -->
+        <update_rate>10</update_rate>
+        <ray>
+          <scan>
+            <horizontal>
+              <samples>500</samples>
+              <resolution>1</resolution>
+              <min_angle>${-pi}</min_angle>
+              <max_angle>${pi}</max_angle>
+            </horizontal>
+            <vertical>
+              <samples>1</samples>
+              <resolution>0.01</resolution>
+              <min_angle>0</min_angle>
+              <max_angle>0</max_angle>
+            </vertical>
+          </scan>
+          <range>
+            <min>0.03</min>
+            <max>12.0</max>
+            <resolution>0.01</resolution>
+          </range>
+          <noise>
+            <!-- +/- 20 mm @ 0.5-2m STD 4mm -->
+            <mean>0.020</mean>
+            <stddev>0.004</stddev>
+          </noise>
+        </ray>
+        <always_on>1</always_on>
+        <visualize>true</visualize>
+      </sensor>
+    </gazebo>
+    <link name="base_link/gpu_lidar" />
+    <joint name="gpu_lidar_joint" type="fixed">
+      <parent link="laser_link" />
+      <child link="base_link/gpu_lidar" />
+    </joint>
+  </xacro:if>
 </robot>

File: brum_description/urdf/sensor_plate.urdf.xacro (robot description, xacro)
@@ -4,10 +4,12 @@
   <xacro:property name="sensor_plate_main_width" value="0.10" />
   <xacro:property name="sensor_plate_main_x_offset" value="-0.0125" />
-  <xacro:property name="sensor_plate_wall_inset" value="-0.002"/>
-  <xacro:property name="sensor_plate_pillar_radius" value="0.002"/>
-  <xacro:property name="sensor_plate_pillar_length" value="0.02"/>
-  <xacro:property name="sensor_plate_chin_thickness" value="0.003"/>
-  <xacro:property name="sensor_plate_chin_length" value="0.012"/>
-  <xacro:property name="sensor_plate_chin_width" value="0.045"/>
+  <xacro:property name="sensor_plate_wall_inset" value="-0.002" />
+  <xacro:property name="sensor_plate_pillar_radius" value="0.002" />
+  <xacro:property name="sensor_plate_pillar_length" value="0.02" />
+  <xacro:property name="sensor_plate_chin_thickness" value="0.003" />
+  <xacro:property name="sensor_plate_chin_length" value="0.012" />
+  <xacro:property name="sensor_plate_chin_width" value="0.045" />
+  <xacro:property name="center_sonar_spread_angle_horizontal" value="${radians(21)}" />
+  <xacro:property name="center_sonar_spread_angle_vertical" value="${radians(4)}" />
   <link name="sensor_plate_link">
     <inertial>
@@ -31,5 +33,6 @@
     </visual>
     <collision name="plate_main">
-      <origin xyz="${sensor_plate_main_width/2+sensor_plate_main_x_offset} 0.0 ${-sensor_plate_main_length/2}"/>
+      <origin
+        xyz="${sensor_plate_main_width/2+sensor_plate_main_x_offset} 0.0 ${-sensor_plate_main_length/2}" />
       <geometry>
         <box size="${sensor_plate_main_width} ${sensor_plate_height} ${sensor_plate_main_length}" />
@@ -37,21 +40,25 @@
     </collision>
     <collision name="plate_pillar_left">
-      <origin xyz="${sensor_plate_main_x_offset-sensor_plate_wall_inset+sensor_plate_pillar_radius} ${sensor_plate_height/2+sensor_plate_pillar_length/2} ${sensor_plate_wall_inset-sensor_plate_pillar_radius}"
-      rpy="${radians(90)} ${radians(90)} 0.0"/>
+      <origin
+        xyz="${sensor_plate_main_x_offset-sensor_plate_wall_inset+sensor_plate_pillar_radius} ${sensor_plate_height/2+sensor_plate_pillar_length/2} ${sensor_plate_wall_inset-sensor_plate_pillar_radius}"
+        rpy="${radians(90)} ${radians(90)} 0.0" />
       <geometry>
-        <cylinder radius="${sensor_plate_pillar_radius}" length="${sensor_plate_pillar_length}"/>
+        <cylinder radius="${sensor_plate_pillar_radius}" length="${sensor_plate_pillar_length}" />
       </geometry>
     </collision>
     <collision name="plate_pillar_right">
-      <origin xyz="${sensor_plate_main_width+sensor_plate_main_x_offset+sensor_plate_wall_inset-sensor_plate_pillar_radius} ${sensor_plate_height/2+sensor_plate_pillar_length/2} ${sensor_plate_wall_inset-sensor_plate_pillar_radius}"
-      rpy="${radians(90)} ${radians(90)} 0.0"/>
+      <origin
+        xyz="${sensor_plate_main_width+sensor_plate_main_x_offset+sensor_plate_wall_inset-sensor_plate_pillar_radius} ${sensor_plate_height/2+sensor_plate_pillar_length/2} ${sensor_plate_wall_inset-sensor_plate_pillar_radius}"
+        rpy="${radians(90)} ${radians(90)} 0.0" />
       <geometry>
-        <cylinder radius="${sensor_plate_pillar_radius}" length="${sensor_plate_pillar_length}"/>
+        <cylinder radius="${sensor_plate_pillar_radius}" length="${sensor_plate_pillar_length}" />
       </geometry>
     </collision>
     <collision>
-      <origin xyz="${sensor_plate_main_width/2+sensor_plate_main_x_offset} ${sensor_plate_chin_thickness/2} ${sensor_plate_chin_length/2}"/>
+      <origin
+        xyz="${sensor_plate_main_width/2+sensor_plate_main_x_offset} ${sensor_plate_chin_thickness/2} ${sensor_plate_chin_length/2}" />
       <geometry>
-        <box size="${sensor_plate_chin_width} ${sensor_plate_chin_thickness} ${sensor_plate_chin_length}"/>
+        <box
+          size="${sensor_plate_chin_width} ${sensor_plate_chin_thickness} ${sensor_plate_chin_length}" />
       </geometry>
     </collision>
@@ -121,3 +128,47 @@
     <child link="center_sonar_link" />
   </joint>
+  <xacro:if value="${mode.startswith('gz-sim')}">
+    <gazebo reference="center_sonar_link">
+      <sensor name='sonar' type='gpu_lidar'>
+        <!-- <pose relative_to='brum/center_sonar_link'>0 0 0 0 0 0</pose> -->
+        <!-- FIXME MAKE RELATIVE TO NAME  -->
+        <topic>/model/brum/sonar_scan</topic>
+        <!-- <frame_id>brum/center_sonar_link</frame_id> -->
+        <update_rate>20</update_rate>
+        <ray>
+          <scan>
+            <horizontal>
+              <samples>25</samples>
+              <resolution>1</resolution>
+              <min_angle>${-center_sonar_spread_angle_horizontal/2}</min_angle>
+              <max_angle>${center_sonar_spread_angle_horizontal/2}</max_angle>
+            </horizontal>
+            <vertical>
+              <samples>25</samples>
+              <resolution>1</resolution>
+              <min_angle>${-center_sonar_spread_angle_vertical/3}</min_angle>
+              <max_angle>${center_sonar_spread_angle_vertical/3}</max_angle>
+            </vertical>
+          </scan>
+          <range>
+            <min>0.02</min>
+            <max>4.0</max>
+            <resolution>0.03</resolution>
+          </range>
+          <!-- https://forum.arduino.cc/t/hc-sr04-tests-on-accuracy-precision-and-resolution-of-ultrasonic-measurement/236505 -->
+          <noise>
+            <mean>0.07</mean>
+            <stddev>0.003</stddev>
+          </noise>
+        </ray>
+        <always_on>1</always_on>
+        <visualize>true</visualize>
+      </sensor>
+    </gazebo>
+    <link name="base_link/sonar" />
+    <joint name="sonar_joint" type="fixed">
+      <parent link="center_sonar_link" />
+      <child link="base_link/sonar" />
+    </joint>
+  </xacro:if>
 </robot>

File: brum_description/urdf/wheels.urdf.xacro (robot description, xacro)
@@ -1,5 +1,13 @@
 <robot xmlns:xacro="http://www.ros.org/wiki/xacro">
-  <xacro:property name="wheel_radius" value="0.035"/>
-  <xacro:property name="wheel_width" value="0.025"/>
+  <!-- 0.035 0.0325  -->
+  <xacro:property name="wheel_radius" value="0.034" />
+  <xacro:property name="wheel_width" value="0.025" />
+  <!-- TODO Maybe scale speeds and torque back to mimic real limitations better -->
+  <!-- 160 RPM @ 6V (https://wiki.dfrobot.com/Micro_DC_Motor_with_Encoder-SJ01_SKU__FIT0450) -->
+  <xacro:property name="max_rotational_velocity_wheel" value="${(160*60)*pi*2}" />
+  <xacro:property name="wheel_separation" value="${0.158-wheel_width}" />
+  <!-- 0.8kgf.cm Max Stall torque
+  (https://wiki.dfrobot.com/Micro_DC_Motor_with_Encoder-SJ01_SKU__FIT0450) -->
+  <xacro:property name="max_wheel_torque" value="0.0784532" />
   <material name="wheel_material">
     <!-- <color rgba="0.79216 0.81961 0.93333 1" /> -->
@@ -22,10 +30,10 @@
         <mesh filename="package://brum_description/meshes/left_wheel.STL" />
       </geometry>
-      <material name="wheel_material"/>
+      <material name="wheel_material" />
     </visual>
     <collision>
-      <origin xyz="0.0 0.0 -${wheel_width/2}"/>
+      <origin xyz="0.0 0.0 -${wheel_width/2}" />
       <geometry>
-        <cylinder radius="${wheel_radius}" length="${wheel_width}"/>
+        <cylinder radius="${wheel_radius}" length="${wheel_width}" />
       </geometry>
     </collision>
@@ -48,10 +56,10 @@
         <mesh filename="package://brum_description/meshes/right_wheel.STL" />
       </geometry>
-      <material name="wheel_material"/>
+      <material name="wheel_material" />
     </visual>
     <collision>
-      <origin xyz="0.0 0.0 ${-wheel_width/2}"/>
+      <origin xyz="0.0 0.0 ${-wheel_width/2}" />
       <geometry>
-        <cylinder radius="${wheel_radius}" length="${wheel_width}"/>
+        <cylinder radius="${wheel_radius}" length="${wheel_width}" />
       </geometry>
     </collision>
@@ -64,4 +72,5 @@
     <child link="left_wheel" />
     <axis xyz="0 0 1" />
+    <limit effort="${max_wheel_torque}" velocity="${max_rotational_velocity_wheel}" />
   </joint>
   <joint name="right_wheel_joint" type="continuous">
@@ -72,4 +81,21 @@
     <child link="right_wheel" />
     <axis xyz="0 0 -1" />
+    <limit effort="${max_wheel_torque}" velocity="${max_rotational_velocity_wheel}" />
   </joint>
+  <xacro:if value="${mode == 'gz-sim-diff-drive-plugin'}">
+    <gazebo>
+      <plugin filename="gz-sim-diff-drive-system" name="gz::sim::systems::DiffDrive">
+        <left_joint>left_wheel_joint</left_joint>
+        <right_joint>right_wheel_joint</right_joint>
+        <wheel_separation>${wheel_separation}</wheel_separation>
+        <wheel_radius>${wheel_radius}</wheel_radius>
+        <!-- Match the ros2_control rate -->
+        <odom_publish_frequency>50</odom_publish_frequency>
+        <max_linear_velocity>${max_rotational_velocity_wheel*wheel_radius}</max_linear_velocity>
+        <min_linear_velocity>${-max_rotational_velocity_wheel*wheel_radius}</min_linear_velocity>
+        <max_angular_velocity>${max_rotational_velocity_wheel*wheel_radius/(wheel_separation/2)}</max_angular_velocity>
+        <min_angular_velocity>${-max_rotational_velocity_wheel*wheel_radius/(wheel_separation/2)}</min_angular_velocity>
+      </plugin>
+    </gazebo>
+  </xacro:if>
 </robot>
